Commit message: limit angle lidar, connect ps4

File: src/amr_reality_pkg/descriptions/urdf/AMR1-00-Khung (1).SLDASM.urdf (robot description, URDF)
Before this commit: robot AMR1-00-Khung (1).SLDASM, 9 links, 8 joints
Joints:
- joint Lidar_Joint: origin xyz=0.33888 -0.00043528 0.12467 rpy=0 0 0 -> xyz=0.33888 -0.00043528 0.12467 rpy=0 0 -1.5708

File: src/amr_reality_pkg/descriptions/urdf/robot.urdf.xacro (robot description, xacro)
@@ -2,6 +2,8 @@
 <robot xmlns:xacro="http://www.ros.org/wiki/xacro" name="my_diff_robot">
     <xacro:include filename="AMR1-00-Khung (1).SLDASM.urdf" />
-    <!-- <xacro:include filename="gazebo_control.xacro" /> -->
-    <!-- <xacro:include filename="sensors.xacro" /> -->
     <xacro:include filename="robot_controller/robot_controller.urdf.xacro" />
+    <!-- <xacro:include filename="gazebo_control.xacro" />
+    <xacro:include filename="sensors.xacro" /> -->
+    <!-- <xacro:include filename="$(find amr_reality_pkg)/descriptions/urdf/robot_controller/AMR1-00-Khung (1).SLDASM.urdf" />
+    <xacro:include filename="$(find amr_reality_pkg)/descriptions/urdf/robot_controller/robot_controller.urdf.xacro" /> -->
 </robot>

File: src/amr_sim_pkg/descriptions/urdf/robot.urdf.xacro (robot description, xacro)
@@ -1,6 +1,6 @@
 <?xml version="1.0"?>
-<robot xmlns:xacro="http://www.ros.org/wiki/xacro" name="my_diff_robot">
-    <xacro:include filename="robot_core.xacro" />
-    <xacro:include filename="gazebo_control.xacro" />
-    <xacro:include filename="sensors.xacro" />
+<robot xmlns:xacro="http://www.ros.org/wiki/xacro" name="my_sim_robot">
+    <xacro:include filename="$(find amr_sim_pkg)/descriptions/urdf/robot_core.xacro" />
+    <xacro:include filename="$(find amr_sim_pkg)/descriptions/urdf/gazebo_control.xacro" />
+    <xacro:include filename="$(find amr_sim_pkg)/descriptions/urdf/sensors.xacro" />
 </robot>

File: src/amr_sim_pkg/descriptions/urdf/sensors.xacro (robot description, xacro)
@@ -3,8 +3,8 @@
     <joint name="laser_joint" type="fixed">
         <parent link="chassis"/>
-        <child link="laser_frame"/>
+        <child link="Lidar_Link"/>
         <origin xyz="0.15 0 0.175" rpy="0 0 0"/>
     </joint>
-    <link name="laser_frame">
+    <link name="Lidar_Link">
         <visual>
             <origin xyz="0 0 0" rpy="0 0 0"/>
@@ -20,5 +20,5 @@
         </xacro:inertial_cylinder>
     </link>
-    <gazebo reference="laser_frame">
+    <!-- <gazebo reference="Lidar_Link">
         <material>Gazebo/Red</material>
         <sensor name="laser" type="ray">
@@ -44,9 +44,9 @@
                 </ros>
                 <output_type>sensor_msgs/LaserScan</output_type>
-                <frame_name>laser_frame</frame_name>
+                <frame_name>Lidar_Link</frame_name>
             </plugin>
         </sensor>
-    </gazebo>
-    <joint name="camera_joint" type="fixed">
+    </gazebo> -->
+    <!-- <joint name="camera_joint" type="fixed">
         <parent link="chassis"/>
         <child link="camera_link"/>
@@ -86,4 +86,4 @@
             </plugin>
         </sensor>
-    </gazebo>
+    </gazebo> -->
 </robot>

Commit message: fix co dinh id cac device, fuse imu encoder_xac dinh chinh xac gox yaw ke ca khi robot truot banh

File: src/amr_reality_pkg/descriptions/urdf/AMR1-00-Khung (1).SLDASM.urdf (robot description, URDF)
Before this commit: robot AMR1-00-Khung (1).SLDASM, 9 links, 8 joints
Links:
- added link Imu_Link, mass 0.0811739569825906; collision mesh filename=file://$(find amr_reality_pkg)/descriptions/meshes/Imu_Link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; visual mesh filename=file://$(find amr_reality_pkg)/descriptions/meshes/Imu_Link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
- link Left_Link: mass 0.663463916376757 -> 0.575934835821199
- link Lidar_Link: mass 0.22083577503254 -> 0.22083577563192
- link Right_Link: mass 0.663463916376758 -> 0.5759348358212
- link Yaw_Behind_Right_Link: mass 0.317263848923435 -> 0.317263848923434
- link Yaw_Front_Right_Link: mass 0.317263848923433 -> 0.317263848923435
- link base_link: mass 10.4160319881205 -> 10.4778859038141
Joints:
- added joint Imu_Joint: type fixed, parent base_link, child Imu_Link, origin xyz=-0.032882 0 0.03125 rpy=0 0 0, axis 0 0 0
- joint Left_Joint: axis 0 1 0 -> 0 -1 0; origin xyz=0.00086753 0.2555 0.055465 rpy=0 0 0 -> xyz=0.0008675297542593 0.2555 0.0554645048190108 rpy=0 0 0
- joint Lidar_Joint: origin xyz=0.33888 -0.00043528 0.12467 rpy=0 0 -1.5708 -> xyz=0.338876449328432 -0.000435283144085308 0.124668485945723 rpy=0 0 -1.5708
- joint Right_Joint: origin xyz=0.00086753 -0.2555 0.055465 rpy=0 0 0 -> xyz=0.000867529754257412 -0.2555 0.0554645048190089 rpy=0 0 0
- joint Yaw_Behind_Left_Joint: axis 0 0 -1 -> 0 0 0; origin xyz=-0.29488 0.199 0.076436 rpy=0 0 0 -> xyz=-0.294882470245741 0.199 0.0764358974358974 rpy=0 0 0
- joint Yaw_Behind_Right_Joint: axis 0 0 -1 -> 0 0 0; origin xyz=-0.29488 -0.199 0.076436 rpy=0 0 0 -> xyz=-0.294882470245742 -0.199 0.0764358974358977 rpy=0 0 0
- joint Yaw_Front_Left_Joint: axis 0 0 -1 -> 0 0 0; origin xyz=0.29512 0.199 0.076436 rpy=0 0 0 -> xyz=0.295117529754259 0.199 0.0764358974358974 rpy=0 0 0
- joint Yaw_Front_Right_Joint: axis 0 0 -1 -> 0 0 0; origin xyz=0.29512 -0.199 0.076436 rpy=0 0 0 -> xyz=0.295117529754259 -0.199000000000001 0.0764358974358964 rpy=0 0 0

File: src/amr_sim_pkg/descriptions/urdf/robot_core.xacro (robot description, xacro)
@@ -5,11 +5,11 @@
     <material name="blue"><color rgba="0 0 1 1"/></material>
     <material name="black"><color rgba="0 0 0 1"/></material>
-    <link name="base_link"></link>
-    <joint name="chassis_joint" type="fixed">
-        <parent link="base_link"/>
-        <child link="chassis"/>
+    <link name="base_footprint"></link>
+    <joint name="base_link_joint" type="fixed">
+        <parent link="base_footprint"/>
+        <child link="base_link"/>
         <origin xyz="0 0 0.075" rpy="0 0 0"/>
     </joint>
-    <link name="chassis">
+    <link name="base_link">
         <visual>
             <origin xyz="0 0 0.075" rpy="0 0 0"/>
@@ -25,7 +25,7 @@
         </xacro:inertial_box>
     </link>
-    <gazebo reference="chassis"><material>Gazebo/White</material></gazebo>
+    <gazebo reference="base_link"><material>Gazebo/White</material></gazebo>
     <joint name="left_wheel_joint" type="continuous">
-        <parent link="chassis"/>
+        <parent link="base_link"/>
         <child link="left_wheel"/>
         <origin xyz="0 0.175 0" rpy="${-pi/2} 0 0"/>
@@ -35,12 +35,12 @@
         <visual>
             <origin xyz="0 0 0" rpy="0 0 0"/>
-            <geometry><cylinder radius="0.05" length="0.04"/></geometry>
+            <geometry><cylinder radius="0.05" length="0.05"/></geometry>
             <material name="blue"/>
         </visual>
         <collision>
             <origin xyz="0 0 0" rpy="0 0 0"/>
-            <geometry><cylinder radius="0.05" length="0.04"/></geometry>
+            <geometry><cylinder radius="0.05" length="0.05"/></geometry>
         </collision>
-        <xacro:inertial_cylinder mass="0.1" length="0.04" radius="0.05">
+        <xacro:inertial_cylinder mass="0.1" length="0.05" radius="0.05">
             <origin xyz="0 0 0" rpy="0 0 0"/>
         </xacro:inertial_cylinder>
@@ -48,5 +48,5 @@
     <gazebo reference="left_wheel"><material>Gazebo/Blue</material></gazebo>
     <joint name="right_wheel_joint" type="continuous">
-        <parent link="chassis"/>
+        <parent link="base_link"/>
         <child link="right_wheel"/>
         <origin xyz="0 -0.175 0" rpy="${pi/2} 0 0"/>
@@ -56,12 +56,12 @@
         <visual>
             <origin xyz="0 0 0" rpy="0 0 0"/>
-            <geometry><cylinder radius="0.05" length="0.04"/></geometry>
+            <geometry><cylinder radius="0.05" length="0.05"/></geometry>
             <material name="blue"/>
         </visual>
         <collision>
             <origin xyz="0 0 0" rpy="0 0 0"/>
-            <geometry><cylinder radius="0.05" length="0.04"/></geometry>
+            <geometry><cylinder radius="0.05" length="0.05"/></geometry>
         </collision>
-        <xacro:inertial_cylinder mass="0.1" length="0.04" radius="0.05">
+        <xacro:inertial_cylinder mass="0.1" length="0.05" radius="0.05">
             <origin xyz="0 0 0" rpy="0 0 0"/>
         </xacro:inertial_cylinder>
@@ -69,5 +69,5 @@
     <gazebo reference="right_wheel"><material>Gazebo/Blue</material></gazebo>
     <joint name="caster_wheel_joint" type="fixed">
-        <parent link="chassis"/>
+        <parent link="base_link"/>
         <child link="caster_wheel"/>
         <origin xyz="0.18 0 0" rpy="0 0 0"/>
@@ -89,6 +89,6 @@
     <gazebo reference="caster_wheel">
         <material>Gazebo/Black</material>
-        <mu1 value="0.001"/>
-        <mu2 value="0.001"/>
+        <mu1 value="0.3"/>
+        <mu2 value="0.3"/>
     </gazebo>
 </robot>

File: src/amr_sim_pkg/descriptions/urdf/sensors.xacro (robot description, xacro)
@@ -2,5 +2,5 @@
 <robot xmlns:xacro="http://www.ros.org/wiki/xacro">
     <joint name="laser_joint" type="fixed">
-        <parent link="chassis"/>
+        <parent link="base_link"/>
         <child link="Lidar_Link"/>
         <origin xyz="0.15 0 0.175" rpy="0 0 0"/>
@@ -20,5 +20,5 @@
         </xacro:inertial_cylinder>
     </link>
-    <!-- <gazebo reference="Lidar_Link">
+    <gazebo reference="Lidar_Link">
         <material>Gazebo/Red</material>
         <sensor name="laser" type="ray">
@@ -47,7 +47,62 @@
             </plugin>
         </sensor>
-    </gazebo> -->
+    </gazebo>
+    <joint name="imu_joint" type="fixed">
+        <parent link ="base_link"/>
+        <child link="imu_link"/>
+        <origin xyz="0.0 0 0.175" rpy="0 0 0"/>
+    </joint>
+    <link name="imu_link">
+        <visual>
+            <origin xyz="0 0 0" rpy="0 0 0"/>
+            <geometry><cylinder radius="0.02" length="0.02"/></geometry>
+            <material name="orange"/>
+        </visual>
+        <collision>
+            <origin xyz="0 0 0" rpy="0 0 0"/>
+            <geometry><cylinder radius="0.02" length="0.02"/></geometry>
+        </collision>
+        <xacro:inertial_cylinder mass="0.04" length="0.02" radius="0.02">
+            <origin xyz="0 0 0" rpy="0 0 0"/>
+        </xacro:inertial_cylinder>
+    </link>
+    <!-- Cấu hình Gazebo cho IMU Sensor -->
+    <gazebo reference="imu_link">
+        <gravity>true</gravity>
+        <sensor name="imu_sensor" type="imu">
+            <always_on>true</always_on>
+            <update_rate>50</update_rate> <!-- Tần số phát dữ liệu (Hz) -->
+            <visualize>true</visualize>
+            <topic>imu</topic>
+            <plugin name="imu_plugin" filename="libgazebo_ros_imu_sensor.so">
+                <ros>
+                    <!-- Remap topic mặc định ra topic IMU chuẩn của ROS 2 -->
+                    <remapping>~/out:=imu/data</remapping>
+                </ros>
+                <!-- Giữ đúng imu_link để TF Tree liên tục -->
+                <frame_name>imu_link</frame_name>
+                <initial_orientation_as_reference>false</initial_orientation_as_reference>
+            </plugin>
+            <!-- <pose>0 0 0 0 0 0</pose> -->
+            <!-- <orientation>
+                <x><noise type="gaussian"><mean>0.0</mean><stddev>0.01</stddev></noise></x>
+                <y><noise type="gaussian"><mean>0.0</mean><stddev>0.01</stddev></noise></y>
+                <z><noise type="gaussian"><mean>0.0</mean><stddev>0.01</stddev></noise></z>
+            </orientation>
+            <angular_velocity>
+                <x><noise type="gaussian"><mean>0.0</mean><stddev>0.001</stddev></noise></x>
+                <y><noise type="gaussian"><mean>0.0</mean><stddev>0.001</stddev></noise></y>
+                <z><noise type="gaussian"><mean>0.0</mean><stddev>0.001</stddev></noise></z>
+            </angular_velocity>
+            <linear_acceleration>
+                <x><noise type="gaussian"><mean>0.0</mean><stddev>0.05</stddev></noise></x>
+                <y><noise type="gaussian"><mean>0.0</mean><stddev>0.05</stddev></noise></y>
+                <z><noise type="gaussian"><mean>0.0</mean><stddev>0.05</stddev></noise></z>
+            </linear_acceleration> -->
+        </sensor>
+        <material>Gazebo/Orange</material>
+    </gazebo>
     <!-- <joint name="camera_joint" type="fixed">
-        <parent link="chassis"/>
+        <parent link="base_link"/>
         <child link="camera_link"/>
         <origin xyz="0.305 0 0.08" rpy="0 0 0"/>
